Commit message: .

File: assets/robot.urdf (robot description, URDF)
Before this commit: robot folderv2, 27 links, 26 joints
Joints:
- joint index_actual_tip_joint: origin xyz=-0.022 0 -0.004 rpy=0 0 0 -> xyz=-0.017 0 -0.004 rpy=0 0 0
- joint index_splay: axis 0 0 -1 -> 0 0 1; limit lower=-0.261799 upper=0.201799 effort=10 velocity=10 -> lower=-0.191799 upper=0.201799 effort=10 velocity=10
- joint middle_actual_tip_joint: origin xyz=-0.02 0.002 -0.004 rpy=0 0 0 -> xyz=-0.015 0.002 -0.004 rpy=0 0 0
- joint pinky_actual_tip_joint: origin xyz=-0.017 0.002 -0.004 rpy=0 0 0 -> xyz=-0.012 0.002 -0.004 rpy=0 0 0
- joint pinky_splay: axis 0 0 -1 -> 0 0 1; limit lower=-0.298132 upper=0.298132 effort=10 velocity=10 -> lower=-0.298132 upper=0.598132 effort=10 velocity=10
- joint ring_actual_tip_joint: origin xyz=-0.02 0.002 -0.004 rpy=0 0 0 -> xyz=-0.015 0.002 -0.004 rpy=0 0 0
- joint ring_splay: axis 0 0 -1 -> 0 0 1; limit lower=-0.301426 upper=0.201426 effort=10 velocity=10 -> lower=-0.301426 upper=0.301426 effort=10 velocity=10

Commit message: .

File: assets/robot.urdf (robot description, URDF)
Before this commit: robot folderv2, 27 links, 26 joints
Joints:
- joint index_actual_tip_joint: origin xyz=-0.017 0 -0.004 rpy=0 0 0 -> xyz=-0.007 0 -0.004 rpy=0 0 0
- joint middle_actual_tip_joint: origin xyz=-0.015 0.002 -0.004 rpy=0 0 0 -> xyz=-0.005 0.002 -0.004 rpy=0 0 0
